File: HW/Electronics/UFOControlDeck/UFOControlDeck.kicad_pcb (KiCad board)
At the start: 4 copper layers, 46 x 46 mm, 84 parts, among them J1 Conn_01x02_Male, J10 Conn_01x02_Male, J13 Conn_02x08_Odd_Even, J2 Conn_02x08_Odd_Even, J3 Conn_01x02_Male, U2 SN74LV1T34DBV, U3 LCMXO3D-4300ZC-3SG72I, U4 ASDMB-xxxMHz, U5 SN74LV1T34DBV, U6 NCP1117-3.3_SOT223, U8 RPX-1.5-tony_bits, U9 LTC6752xUD-3

Commit message: files for manufactured mothership pulsedeck and controldeck
Parts:
- removed J10, J3: Conn_01x02_Male, Connector_PinHeader_1.27mm:PinHeader_1x02_P1.27mm_Vertical
- removed RV1: R_POT, Potentiometer_SMD:Potentiometer_Bourns_3214W_Vertical
- added J4: Conn_Coaxial, Connector_Coaxial:U.FL_Hirose_U.FL-R-SMT-1_Vertical, B.Cu at (139.4, 99.4)
- added J5: Conn_Coaxial, Connector_Coaxial:U.FL_Hirose_U.FL-R-SMT-1_Vertical, F.Cu at (157.2, 107.0)
- added J6: Conn_Coaxial, Connector_Coaxial:U.FL_Hirose_U.FL-R-SMT-1_Vertical, B.Cu at (156.8, 106.7)
- added R27: 0r, Resistor_SMD:R_0603_1608Metric_Pad0.98x0.95mm_HandSolder, F.Cu at (133.8, 104.5)
- added R28: DNF, Resistor_SMD:R_0603_1608Metric_Pad0.98x0.95mm_HandSolder, F.Cu at (132.3, 104.5)
- added U1: ADR4530, Package_SO:SOIC-8_3.9x4.9mm_P1.27mm, B.Cu at (132.8, 103.5)
- moved C11 3.79 mm to (139.1, 103.1), turned to -90 degrees
Connections:
- net +3V3 renamed +3.3V
- net /~Q renamed /~{Q}
- H1 pad 1: Net-(H1-Pad1) -> unconnected-(H1-Pad1)
- H2 pad 1: Net-(H2-Pad1) -> unconnected-(H2-Pad1)
- H3 pad 1: Net-(H3-Pad1) -> unconnected-(H3-Pad1)
- H4 pad 1: Net-(H4-Pad1) -> unconnected-(H4-Pad1)
- J2 pad 1: Net-(J2-Pad1) -> unconnected-(J2-Pad1)
- J2 pad 10: Net-(J2-Pad10) -> unconnected-(J2-Pad10)
- J2 pad 12: Net-(J2-Pad12) -> unconnected-(J2-Pad12)
- J2 pad 14: Net-(J2-Pad14) -> unconnected-(J2-Pad14)
- J2 pad 16: Net-(J2-Pad16) -> unconnected-(J2-Pad16)
- J2 pad 2: Net-(J2-Pad2) -> unconnected-(J2-Pad2)
- J2 pad 3: Net-(J2-Pad3) -> unconnected-(J2-Pad3)
- J2 pad 4: Net-(J2-Pad4) -> unconnected-(J2-Pad4)
- J2 pad 5: Net-(J2-Pad5) -> unconnected-(J2-Pad5)
- J2 pad 6: Net-(J2-Pad6) -> unconnected-(J2-Pad6)
- J2 pad 8: Net-(J2-Pad8) -> unconnected-(J2-Pad8)
- R2 pad 1: ~COMP -> ~{COMP}
- U2 pad 1: Net-(U2-Pad1) -> unconnected-(U2-Pad1)
- U3 pad 14: Net-(U3-Pad14) -> unconnected-(U3-Pad14)
- U3 pad 16: Net-(U3-Pad16) -> unconnected-(U3-Pad16)
- U3 pad 17: Net-(U3-Pad17) -> unconnected-(U3-Pad17)
- U3 pad 19: Net-(U3-Pad19) -> unconnected-(U3-Pad19)
- U3 pad 20: Net-(U3-Pad20) -> unconnected-(U3-Pad20)
- U3 pad 21: Net-(U3-Pad21) -> unconnected-(U3-Pad21)
- U3 pad 22: Net-(U3-Pad22) -> unconnected-(U3-Pad22)
- U3 pad 24: Net-(U3-Pad24) -> unconnected-(U3-Pad24)
- U3 pad 26: Net-(U3-Pad26) -> COMP
- U3 pad 27: Net-(U3-Pad27) -> TRIGGER
- U3 pad 28: Net-(U3-Pad28) -> unconnected-(U3-Pad28)
- U3 pad 3: Net-(U3-Pad3) -> unconnected-(U3-Pad3)
- U3 pad 30: Net-(U3-Pad30) -> unconnected-(U3-Pad30)
- U3 pad 31: Net-(U3-Pad31) -> unconnected-(U3-Pad31)
- U3 pad 33: Net-(U3-Pad33) -> unconnected-(U3-Pad33)
- U3 pad 34: Net-(U3-Pad34) -> unconnected-(U3-Pad34)
- U3 pad 35: Net-(U3-Pad35) -> unconnected-(U3-Pad35)
- U3 pad 36: Net-(U3-Pad36) -> unconnected-(U3-Pad36)
- U3 pad 37: COMP -> unconnected-(U3-Pad37)
- U3 pad 38: TRIGGER -> unconnected-(U3-Pad38)
- U3 pad 4: Net-(U3-Pad4) -> unconnected-(U3-Pad4)
- U3 pad 40: Net-(U3-Pad40) -> unconnected-(U3-Pad40)
- U3 pad 41: Net-(U3-Pad41) -> ~{COMP}
- U3 pad 43: Net-(U3-Pad43) -> ~{TRIGGER}
- U3 pad 44: Net-(U3-Pad44) -> unconnected-(U3-Pad44)
- U3 pad 45: Net-(U3-Pad45) -> unconnected-(U3-Pad45)
- U3 pad 47: Net-(U3-Pad47) -> unconnected-(U3-Pad47)
- U3 pad 49: Net-(U3-Pad49) -> unconnected-(U3-Pad49)
- U3 pad 50: Net-(U3-Pad50) -> unconnected-(U3-Pad50)
- U3 pad 51: ~TRIGGER -> unconnected-(U3-Pad51)
- U3 pad 52: ~COMP -> unconnected-(U3-Pad52)
- U3 pad 53: Net-(U3-Pad53) -> unconnected-(U3-Pad53)
- U3 pad 56: Net-(U3-Pad56) -> unconnected-(U3-Pad56)
- U3 pad 57: Net-(U3-Pad57) -> unconnected-(U3-Pad57)
- U3 pad 58: Net-(U3-Pad58) -> unconnected-(U3-Pad58)
- U3 pad 59: Net-(U3-Pad59) -> unconnected-(U3-Pad59)
- U3 pad 63: Net-(U3-Pad63) -> unconnected-(U3-Pad63)
- U3 pad 65: Net-(U3-Pad65) -> unconnected-(U3-Pad65)
- U3 pad 66: Net-(U3-Pad66) -> unconnected-(U3-Pad66)
- U3 pad 67: Net-(U3-Pad67) -> unconnected-(U3-Pad67)
- U3 pad 68: Net-(U3-Pad68) -> unconnected-(U3-Pad68)
- U3 pad 69: Net-(U3-Pad69) -> unconnected-(U3-Pad69)
- U5 pad 1: Net-(U5-Pad1) -> unconnected-(U5-Pad1)
- U5 pad 4: ~TRIGGER -> ~{TRIGGER}
- U8 pad 12: Net-(U8-Pad12) -> unconnected-(U8-Pad12)
- U8 pad 6_7_8: Net-(U8-Pad6_7_8) -> unconnected-(U8-Pad6_7_8)
- U9 pad 11: Net-(U9-Pad11) -> unconnected-(U9-Pad11)
- U9 pad 5: Net-(U9-Pad5) -> unconnected-(U9-Pad5)
- U9 pad 7: Net-(U9-Pad7) -> unconnected-(U9-Pad7)
- U9 pad 8: Net-(U9-Pad8) -> unconnected-(U9-Pad8)
Routing:
- net ~{TRIGGER}: track 0.00 -> 17.0 mm, vias 0 -> 2
- net ~{COMP}: track 0.00 -> 13.9 mm
- net ~TRIGGER: track 13.7 -> 0.00 mm
- net ~COMP: track 9.93 -> 0.00 mm
- net COMP: track 20.8 -> 27.2 mm
- net TRIGGER: track 20.8 -> 26.1 mm
- net GND: track 31.7 -> 27.2 mm, vias 37 -> 43
- net Net-(R27-Pad2): track 0.00 -> 4.45 mm, vias 0 -> 1
- net +3.3V: track 57.1 -> 53.4 mm, vias 30 -> 29
- net PULSE6: track 27.0 -> 29.1 mm
- net Net-(R25-Pad1): track 10.7 -> 8.73 mm
- net PULSE7: track 26.4 -> 28.3 mm
- net Net-(D1-Pad1): track 2.08 -> 3.60 mm
- net Net-(H2-Pad1): track 1.02 -> 0.00 mm
- net Net-(C10-Pad1): track 8.43 -> 9.28 mm, vias 0 -> 1
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Other:
- net class Default removed
- board text added: "UFO Control Deck v0.3"
- board text removed: "UFO Control Deck v0.2"
