File: HW/Electronics/UFOControlDeck/UFOControlDeck.sch (KiCad schematic (older format))
At the start: 104 parts, among them J1 Conn_01x02_Male, J10 Conn_01x02_Male, J13 Conn_02x08_Odd_Even, J2 Conn_02x04_Odd_Even, U1 TPSM84209RKHT, U2 LM555xM, U3 ICE40HX8K-BG121, U4 ASDMB-xxxMHz, U5 SN74LV1T34DBV, U6 MT25QL128ABA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

Commit message: Added control deck Interactive BoM
Parts:
- U1, U7, U8: symbol 2021-02-02_14-31-31:TPSM84209RKHT -> UFOControlDeck-rescue:TPSM84209RKHT-2021-02-02_14-31-31
- U6: symbol ants_bits:MT25QL128ABA -> UFOControlDeck-rescue:MT25QL128ABA-ants_bits
Changed lines of the file:
@@
 	14800 12500 14200 12500
 $Comp
-L ants_bits:MT25QL128ABA U6
+L UFOControlDeck-rescue:MT25QL128ABA-ants_bits U6
 U 1 1 602FC3D3
 P 19550 12850
@@
 	14500 12600 14800 12600
 $Comp
-L 2021-02-02_14-31-31:TPSM84209RKHT U7
+L UFOControlDeck-rescue:TPSM84209RKHT-2021-02-02_14-31-31 U7
 U 1 1 60213ABE
 P 4450 7150
@@
 $EndComp
 $Comp
-L 2021-02-02_14-31-31:TPSM84209RKHT U1
+L UFOControlDeck-rescue:TPSM84209RKHT-2021-02-02_14-31-31 U1
 U 1 1 606DE208
 P 4400 9950
@@
 	6950 9450 6950 9200
 $Comp
-L 2021-02-02_14-31-31:TPSM84209RKHT U8
+L UFOControlDeck-rescue:TPSM84209RKHT-2021-02-02_14-31-31 U8
 U 1 1 6070A73E
 P 4400 12750

Commit message: Starting FPGA part switch to LCMXO3D-4300ZC-3SG72I
Parts:
- removed C41: 47u, Capacitor_SMD:C_0603_1608Metric_Pad1.08x0.95mm_HandSolder, symbol Device:C
- removed J2: Conn_02x04_Odd_Even, Connector_PinHeader_1.27mm:PinHeader_2x04_P1.27mm_Vertical_SMD, symbol Connector_Generic:Conn_02x04_Odd_Even
- removed U1, U7, U8: TPSM84209RKHT, TPSM84209:TPSM84209RKHT, symbol UFOControlDeck-rescue:TPSM84209RKHT-2021-02-02_14-31-31
- removed U2: LM555xM, Package_SO:SOIC-8_3.9x4.9mm_P1.27mm, symbol Timer:LM555xM
- removed U6: MT25QL128ABA, Package_DFN_QFN:DFN-8-1EP_6x5mm_P1.27mm_EP2x2mm, symbol UFOControlDeck-rescue:MT25QL128ABA-ants_bits
- added C49: 50n, Capacitor_SMD:C_0603_1608Metric_Pad1.08x0.95mm_HandSolder, symbol Device:C
- added D2: D_Schottky, Diode_SMD:D_0603_1608Metric_Pad1.05x0.95mm_HandSolder, symbol Device:D_Schottky
- added H1, H2, H3, H4: MountingHole_Pad, MountingHole:MountingHole_4.3mm_M4_DIN965_Pad, symbol Mechanical:MountingHole_Pad
- added J2: Conn_02x08_Counter_Clockwise, Connector_PinSocket_1.27mm:PinSocket_2x08_P1.27mm_Vertical_SMD, symbol Connector_Generic:Conn_02x08_Counter_Clockwise
- added J3: Conn_01x02_Male, Connector_PinHeader_1.27mm:PinHeader_1x02_P1.27mm_Vertical, symbol Connector:Conn_01x02_Male
- added R32: 10k, Resistor_SMD:R_0603_1608Metric_Pad0.98x0.95mm_HandSolder, symbol Device:R
- added R33: 200K, Resistor_SMD:R_0603_1608Metric_Pad0.98x0.95mm_HandSolder, symbol Device:R
- added R34: 142K, Resistor_SMD:R_0603_1608Metric_Pad0.98x0.95mm_HandSolder, symbol Device:R
- added R35: 14.3K, Resistor_SMD:R_0603_1608Metric_Pad0.98x0.95mm_HandSolder, symbol Device:R
- added RV1: R_POT, Potentiometer_SMD:Potentiometer_Bourns_3214W_Vertical, symbol Device:R_POT
- added U1, U7: ADP123, symbol tony_bits:ADP123
- added U2: SN74LV1T34DBV, Package_TO_SOT_SMD:SOT-23-5, symbol Logic_LevelTranslator:SN74LV1T34DBV
- added U6: W25Q128JVS, Package_SO:SOIC-8_5.23x5.23mm_P1.27mm, symbol Memory_Flash:W25Q128JVS
- added U8: RPX-1.5, symbol tony_bits:RPX-1.5
- added U9: LTC6752xUD-3, Package_DFN_QFN:QFN-12-1EP_3x3mm_P0.5mm_EP1.65x1.65mm, symbol Comparator:LTC6752xUD-3
- C1, C5: value 10u -> 1u
- C12: value 10n -> C
- C39, C40, C8, C9: value 47u -> 10u
- C4: value 10u -> 47u
- C7: value 47u -> 1u
- D4: footprint Diode_SMD:D_SOD-123F -> Diode_SMD:D_0603_1608Metric_Pad1.05x0.95mm_HandSolder
- R1: value 10k -> 200K
- R2: value 2.21k -> 35.65K
- R4, R5: value 10k -> 100k
- R6: value 1.37k -> 75K
- R9: value R -> 10k
- U3: digikey# (none) -> 220-2148-ND; manf# (none) -> ICE40HX8K-BG121
- U3: digikey# (none) -> 220-2148-ND
- U3: manf# (none) -> ICE40HX8K-BG121
Connections:
- net labels added: CDONE, CRESET, Q, ~Q, ~TRIGGER
- wire segments 447 -> 475
- no-connect marks 0 -> 7
Other:
- moved on the sheet: C1, C10, C11, C46, C7, D4, J10, R1, R11, R2, R25, R26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

Commit message: pcb and schematic changes for machxo3d
Parts:
- removed C47: C, Capacitor_SMD:C_0603_1608Metric_Pad1.08x0.95mm_HandSolder, symbol Device:C
- removed R25, R26, R27, R28, R29, R30: 10k, Resistor_SMD:R_0603_1608Metric_Pad0.98x0.95mm_HandSolder, symbol Device:R
- removed U3: ICE40HX8K-BG121, Package_BGA:BGA-121_9.0x9.0mm_Layout11x11_P0.8mm_Ball0.4mm_Pad0.35mm_NSMD, symbol FPGA_Lattice:ICE40HX8K-BG121
- removed U6: W25Q128JVS, Package_SO:SOIC-8_5.23x5.23mm_P1.27mm, symbol Memory_Flash:W25Q128JVS
- removed U7: ADP123, symbol tony_bits:ADP123
- added U3: LCMXO3D-4300ZC-3SG72I, Package_DFN_QFN:QFN-72-1EP_10x10mm_P0.5mm_EP6x6mm_ThermalVias, symbol MachXO3D:LCMXO3D-4300ZC-3SG72I
- added U6: NCP1117-3.3_SOT223, Package_TO_SOT_SMD:SOT-223-3_TabPin2, symbol Regulator_Linear:NCP1117-3.3_SOT223
- U1: symbol tony_bits:ADP123 -> UFOControlDeck-rescue:ADP123-tony_bits
- U8: symbol tony_bits:RPX-1.5 -> UFOControlDeck-rescue:RPX-1.5-tony_bits
Connections:
- wire segments 475 -> 447

Commit message: main changes made to swap fpga, comparator and power supplies
Parts:
- removed C15, C16, C17, C18, C19, C20, C21, C22, C23, C24, C25, C26, C27, C28, C29, C36, C42, C43, C44, C45: 100n, Capacitor_SMD:C_0603_1608Metric_Pad1.08x0.95mm_HandSolder, symbol Device:C
- removed C2, C3: 10u, Capacitor_SMD:C_0603_1608Metric_Pad1.08x0.95mm_HandSolder, symbol Device:C
- removed C5: 1u, Capacitor_SMD:C_0603_1608Metric_Pad1.08x0.95mm_HandSolder, symbol Device:C
- removed D14: D_Schottky, Diode_SMD:D_SOD-123F, symbol Device:D_Schottky
- removed J2: Conn_02x08_Counter_Clockwise, Connector_PinSocket_1.27mm:PinSocket_2x08_P1.27mm_Vertical_SMD, symbol Connector_Generic:Conn_02x08_Counter_Clockwise
- removed R31: 2k2, Resistor_SMD:R_0603_1608Metric_Pad0.98x0.95mm_HandSolder, symbol Device:R
- removed R33: 200K, Resistor_SMD:R_0603_1608Metric_Pad0.98x0.95mm_HandSolder, symbol Device:R
- removed R34: 142K, Resistor_SMD:R_0603_1608Metric_Pad0.98x0.95mm_HandSolder, symbol Device:R
- removed U1: ADP123, symbol UFOControlDeck-rescue:ADP123-tony_bits
- added D3: LED, LED_SMD:LED_0603_1608Metric_Pad1.05x0.95mm_HandSolder, symbol Device:LED
- added J2: Conn_02x08_Odd_Even, Connector_PinSocket_1.27mm:PinSocket_2x08_P1.27mm_Vertical_SMD, symbol Connector_Generic:Conn_02x08_Odd_Even
- added R25: 1k, Resistor_SMD:R_0603_1608Metric_Pad0.98x0.95mm_HandSolder, symbol Device:R
- added R26: 10k, Resistor_SMD:R_0603_1608Metric_Pad0.98x0.95mm_HandSolder, symbol Device:R
- C4: value 47u -> 22p
- R1: value 200K -> 0r
- R2: value 35.65K -> 0r
- R3, R9: value 10k -> 1k
- R7: value 100R -> 1k
- R8: value 100R -> 10k
- U3: symbol MachXO3D:LCMXO3D-4300ZC-3SG72I -> UFOControlDeck-rescue:LCMXO3D-4300ZC-3SG72I-MachXO3D
- U8: value RPX-1.5 -> RPX-1.5-tony_bits; footprint (none) -> Recom:CONV_RPX-1.5-R
Connections:
- net labels added: COMP, TCK, TDI, TDO, TMS, ~COMP
- net labels removed: +1V2, CDONE, CRESET, FLASH_WP, HOLD_RST, SCK, SDI, SDO, SS_FLASH
- wire segments 447 -> 331
Other:
- moved on the sheet: C30, C31, C32, C33, C34, C35, C37, C38, D13, R24, U3C, U3D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

Commit message: v0.2 design manufactured but requires fixing drill size and traces as not supported by manufacturer
Connections:
- net DONE: now reaches D13.2 (A), R8.1, U3.54 (PT28D-DONE)
- net INITN: now reaches D1.2 (A), R10.1, U3.55 (PT28C-INITN)
- net PROGRAMN: now reaches D3.2 (A), R26.1, U3.61 (PT23D-PROGRAMN)
Changed lines of the file:
@@
 	-1   0    0    1
 $EndComp
+Text Label 15500 11000 0    50   ~ 0
+DONE
+Text Label 15500 11200 0    50   ~ 0
+INITN
+Text Label 15500 11400 0    50   ~ 0
+PROGRAMN
 $EndSCHEMATC

Commit message: files for manufactured mothership pulsedeck and controldeck
Parts:
- added U1: ADR4530, Package_SO:SOIC-8_3.9x4.9mm_P1.27mm, symbol Reference_Voltage:ADR4530
Connections:
- net labels added: ~{COMP}, ~{Q}, ~{TRIGGER}
- net labels removed: ~COMP, ~Q, ~TRIGGER
- wire segments 331 -> 342
